File: forager-pcb/forager-pcb.kicad_sch (KiCad schematic)
At the start: 76 parts, among them J1 Conn_01x02_Pin, J2 Conn_01x02_Pin

Commit message: Add extra column and remove all traces
Parts:
- added LCH1, LCH13, LCH7, RCH12, RCH18, RCH6: ChocHS, Custom:SW_choc_v1_HS_MBK, symbol Switch:SW_Push_45deg
- added LD1, LD13, LD7, RD12, RD18, RD6: D, Diode_SMD:D_SOD-123, symbol Device:D
- renumbered LCH8 to LCH10, LCH9 to LCH11, LCH10 to LCH12, LCH11 to LCH14, LCH12 to LCH15, LCH13 to LCH16, LCH14 to LCH17, LCH15 to LCH18, LCH16 to LCH19, LCH1 to LCH2, LCH17 to LCH20, LCH2 to LCH3, LCH3 to LCH4, LCH4 to LCH5, LCH5 to LCH6, LCH6 to LCH8, LCH7 to LCH9, LD8 to LD10, LD9 to LD11, LD10 to LD12, LD11 to LD14, LD12 to LD15, LD13 to LD16, LD14 to LD17, LD15 to LD18, LD16 to LD19, LD1 to LD2, LD17 to LD20, LD2 to LD3, LD3 to LD4, LD4 to LD5, LD5 to LD6, LD6 to LD8, LD7 to LD9, RCH9 to RCH10, RCH10 to RCH11, RCH11 to RCH13, RCH12 to RCH14, RCH13 to RCH15, RCH14 to RCH16, RCH15 to RCH17, RCH16 to RCH19, RCH17 to RCH20, RCH6 to RCH7, RCH7 to RCH8, RCH8 to RCH9, RD9 to RD10, RD10 to RD11, RD11 to RD13, RD12 to RD14, RD13 to RD15, RD14 to RD16, RD15 to RD17, RD16 to RD19, RD17 to RD20, RD6 to RD7, RD7 to RD8, RD8 to RD9, TP3 to TP2, TP2 to TP3
Connections:
- net LCOL0: now also LCH1.1, LCH13.1, LCH7.1; no longer LCH14.1, LCH2.1, LCH8.1
- net LCOL1: now also LCH14.1, LCH2.1, LCH8.1; no longer LCH15.1, LCH3.1, LCH9.1
- net LCOL2: now also LCH15.1, LCH3.1, LCH9.1; no longer LCH10.1, LCH16.1, LCH4.1
- net LCOL3: now also LCH10.1, LCH16.1, LCH4.1; no longer LCH11.1, LCH17.1, LCH19.1, LCH5.1
- net LCOL4: now also LCH11.1, LCH17.1, LCH19.1, LCH5.1; no longer LCH12.1, LCH18.1, LCH20.1, LCH6.1
- net LROW0: now also LU1.11 (P1.15/10), LD1.1 (K); no longer LU1.7 (P1.11/6)
- net LROW1: now also LU1.12 (P1.14/9), LD7.1 (K); no longer LU1.13 (P1.13/8)
- net LROW2: now also LU1.13 (P1.13/8), LD13.1 (K); no longer LU1.14 (P1.12/7)
- net LROW3: now also LU1.14 (P1.12/7); no longer LU1.12 (P1.14/9)
- net RCOL0: now also RU1.1 (P0.02/0), RCH12.1, RCH18.1, RCH6.1; no longer RCH11.1, RCH17.1, RCH5.1, RU1.3 (P0.28/2)
- net RCOL1: now also RCH11.1, RCH17.1, RCH5.1, RU1.2 (P0.03/1); no longer RCH10.1, RCH16.1, RCH4.1, RU1.4 (P0.29/3)
- net RCOL2: now also RCH10.1, RCH16.1, RCH4.1, RU1.3 (P0.28/2); no longer RCH15.1, RCH3.1, RCH9.1, RU1.5 (P0.04/4)
- net RCOL3: now also RCH15.1, RCH3.1, RCH9.1, RU1.4 (P0.29/3); no longer RCH14.1, RCH2.1, RCH20.1, RCH8.1, RU1.11 (P1.15/10)
- net RCOL4: now also RCH14.1, RCH2.1, RCH20.1, RCH8.1, RU1.5 (P0.04/4); no longer RCH1.1, RCH13.1, RCH19.1, RCH7.1, RU1.12 (P1.14/9)
- net RROW0: now also RU1.11 (P1.15/10), RD6.1 (K); no longer RU1.14 (P1.12/7)
- net RROW1: now also RU1.12 (P1.14/9), RD12.1 (K); no longer RU1.13 (P1.13/8)
- net RROW2: now also RU1.13 (P1.13/8), RD18.1 (K); no longer RU1.2 (P0.03/1)
- net RROW3: now also RU1.14 (P1.12/7); no longer RU1.1 (P0.02/0)
- net RCOL5: now reaches RU1.6 (P0.05/5)
- net RCOL5: now also RCH1.1, RCH13.1, RCH19.1, RCH7.1
- net LCOL5: now reaches LU1.6 (P0.05/5)
- net LCOL5: now also LCH12.1, LCH18.1, LCH20.1, LCH6.1
- new net: LCH1.2, LD1.2 (A)
- new net: LCH13.2, LD13.2 (A)
- new net: RCH6.2, RD6.2 (A)
- new net: RCH12.2, RD12.2 (A)
- new net: LCH7.2, LD7.2 (A)
- new net: RCH18.2, RD18.2 (A)
Other:
- moved on the sheet: LCH10, LCH11, LCH12, LCH14, LCH15, LCH16, LCH17, LCH18, LCH19, LCH2, LCH20, LCH3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
