File: forager-pcb/forager-pcb.kicad_sch (KiCad schematic)
At the start: 88 parts, among them J1 Conn_01x02_Pin, J2 Conn_01x02_Pin

Commit message: Swap to solder sockets
Parts:
- LCH1, LCH10, LCH11, LCH12, LCH13, LCH14, LCH15, LCH16, LCH17, LCH18, LCH19, LCH2, LCH20, LCH3, LCH4, LCH5, LCH6, LCH7, LCH8, LCH9, RCH1, RCH10, RCH11, RCH12, RCH13, RCH14, RCH15, RCH16, RCH17, RCH18, RCH19, RCH2, RCH20, RCH3, RCH4, RCH5, RCH6, RCH7, RCH8, RCH9: footprint Custom:SW_choc_v1v2_HS_MBK -> Custom:Choc_v2_PG1353_socket
Changed lines of the file:
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@@
 			)
 		)
-		(property "Footprint" "Custom:SW_choc_v1v2_HS_MBK"
+		(property "Footprint" "Custom:Choc_v2_PG1353_socket"
 			(at 236.22 109.22 0)
 			(effects
@@
 			)
 		)
-		(property "Footprint" "Custom:SW_choc_v1v2_HS_MBK"
+		(property "Footprint" "Custom:Choc_v2_PG1353_socket"
 			(at 31.75 90.17 0)
 			(effects
@@
 			)
 		)
-		(property "Footprint" "Custom:SW_choc_v1v2_HS_MBK"
+		(property "Footprint" "Custom:Choc_v2_PG1353_socket"
 			(at 86.36 110.49 0)
 			(effects
@@
 			)
 		)
-		(property "Footprint" "Custom:SW_choc_v1v2_HS_MBK"
+		(property "Footprint" "Custom:Choc_v2_PG1353_socket"
 			(at 236.22 68.58 0)
 			(effects
@@
 			)
 		)
-		(property "Footprint" "Custom:SW_choc_v1v2_HS_MBK"
+		(property "Footprint" "Custom:Choc_v2_PG1353_socket"
 			(at 73.66 90.17 0)
 			(effects
@@
 			)
 		)
-		(property "Footprint" "Custom:SW_choc_v1v2_HS_MBK"
+		(property "Footprint" "Custom:Choc_v2_PG1353_socket"
 			(at 184.15 88.9 0)
 			(effects
@@
 			)
 		)
-		(property "Footprint" "Custom:SW_choc_v1v2_HS_MBK"
+		(property "Footprint" "Custom:Choc_v2_PG1353_socket"
 			(at 46.99 69.85 0)
 			(effects
@@
 			)
 		)
-		(property "Footprint" "Custom:SW_choc_v1v2_HS_MBK"
+		(property "Footprint" "Custom:Choc_v2_PG1353_socket"
 			(at 209.55 109.22 0)
 			(effects
@@
 			)
 		)
-		(property "Footprint" "Custom:SW_choc_v1v2_HS_MBK"
+		(property "Footprint" "Custom:Choc_v2_PG1353_socket"
 			(at 184.15 68.58 0)
 			(effects
@@
 			)
 		)
-		(property "Footprint" "Custom:SW_choc_v1v2_HS_MBK"
+		(property "Footprint" "Custom:Choc_v2_PG1353_socket"
 			(at 73.66 110.49 0)
 			(effects
@@
 			)
 		)
-		(property "Footprint" "Custom:SW_choc_v1v2_HS_MBK"
+		(property "Footprint" "Custom:Choc_v2_PG1353_socket"
 			(at 196.85 68.58 0)
 			(effects
@@
 			)
 		)
-		(property "Footprint" "Custom:SW_choc_v1v2_HS_MBK"
+		(property "Footprint" "Custom:Choc_v2_PG1353_socket"
 			(at 180.34 130.81 0)
 			(effects
@@
 			)
 		)
-		(property "Footprint" "Custom:SW_choc_v1v2_HS_MBK"
+		(property "Footprint" "Custom:Choc_v2_PG1353_socket"
 			(at 209.55 68.58 0)
 			(effects
@@
 			)
 		)
-		(property "Footprint" "Custom:SW_choc_v1v2_HS_MBK"
+		(property "Footprint" "Custom:Choc_v2_PG1353_socket"
 			(at 86.36 90.17 0)
 			(effects
@@
 			)
 		)
-		(property "Footprint" "Custom:SW_choc_v1v2_HS_MBK"
+		(property "Footprint" "Custom:Choc_v2_PG1353_socket"
 			(at 73.66 69.85 0)
 			(effects
@@
 			)
 		)
-		(property "Footprint" "Custom:SW_choc_v1v2_HS_MBK"
+		(property "Footprint" "Custom:Choc_v2_PG1353_socket"
 			(at 60.96 69.85 0)
 			(effects
@@
 			)
 		)
-		(property "Footprint" "Custom:SW_choc_v1v2_HS_MBK"
+		(property "Footprint" "Custom:Choc_v2_PG1353_socket"
 			(at 102.87 132.08 0)
 			(effects
@@
 			)
 		)
-		(property "Footprint" "Custom:SW_choc_v1v2_HS_MBK"
+		(property "Footprint" "Custom:Choc_v2_PG1353_socket"
 			(at 86.36 69.85 0)
 			(effects
@@
 			)
 		)
-		(property "Footprint" "Custom:SW_choc_v1v2_HS_MBK"
+		(property "Footprint" "Custom:Choc_v2_PG1353_socket"
 			(at 236.22 88.9 0)
 			(effects
@@
 			)
 		)
-		(property "Footprint" "Custom:SW_choc_v1v2_HS_MBK"
+		(property "Footprint" "Custom:Choc_v2_PG1353_socket"
 			(at 196.85 88.9 0)
 			(effects
@@
 			)
 		)
-		(property "Footprint" "Custom:SW_choc_v1v2_HS_MBK"
+		(property "Footprint" "Custom:Choc_v2_PG1353_socket"
 			(at 209.55 88.9 0)
 			(effects
@@
 			)
 		)
-		(property "Footprint" "Custom:SW_choc_v1v2_HS_MBK"
+		(property "Footprint" "Custom:Choc_v2_PG1353_socket"
 			(at 222.25 88.9 0)
 			(effects
@@
 			)
 		)
-		(property "Footprint" "Custom:SW_choc_v1v2_HS_MBK"
+		(property "Footprint" "Custom:Choc_v2_PG1353_socket"
 			(at 88.9 132.08 0)
 			(effects
@@
 			)
 		)
-		(property "Footprint" "Custom:SW_choc_v1v2_HS_MBK"
+		(property "Footprint" "Custom:Choc_v2_PG1353_socket"
 			(at 31.75 110.49 0)
 			(effects
@@
 			)
 		)
-		(property "Footprint" "Custom:SW_choc_v1v2_HS_MBK"
+		(property "Footprint" "Custom:Choc_v2_PG1353_socket"
 			(at 99.06 69.85 0)
 			(effects
@@
 			)
 		)
-		(property "Footprint" "Custom:SW_choc_v1v2_HS_MBK"
+		(property "Footprint" "Custom:Choc_v2_PG1353_socket"
 			(at 184.15 109.22 0)
 			(effects
@@
 			)
 		)
-		(property "Footprint" "Custom:SW_choc_v1v2_HS_MBK"
+		(property "Footprint" "Custom:Choc_v2_PG1353_socket"
 			(at 46.99 110.49 0)
 			(effects
@@
 			)
 		)
-		(property "Footprint" "Custom:SW_choc_v1v2_HS_MBK"
+		(property "Footprint" "Custom:Choc_v2_PG1353_socket"
 			(at 250.19 109.22 0)
 			(effects
@@
 			)
 		)
-		(property "Footprint" "Custom:SW_choc_v1v2_HS_MBK"
+		(property "Footprint" "Custom:Choc_v2_PG1353_socket"
 			(at 222.25 109.22 0)
 			(effects
@@
 			)
 		)
-		(property "Footprint" "Custom:SW_choc_v1v2_HS_MBK"
+		(property "Footprint" "Custom:Choc_v2_PG1353_socket"
 			(at 196.85 109.22 0)
 			(effects
@@
 			)
 		)
-		(property "Footprint" "Custom:SW_choc_v1v2_HS_MBK"
+		(property "Footprint" "Custom:Choc_v2_PG1353_socket"
 			(at 250.19 88.9 0)
 			(effects
@@
 			)
 		)
-		(property "Footprint" "Custom:SW_choc_v1v2_HS_MBK"
+		(property "Footprint" "Custom:Choc_v2_PG1353_socket"
 			(at 99.06 90.17 0)
 			(effects
@@
 			)
 		)
-		(property "Footprint" "Custom:SW_choc_v1v2_HS_MBK"
+		(property "Footprint" "Custom:Choc_v2_PG1353_socket"
 			(at 222.25 68.58 0)
 			(effects
@@
 			)
 		)
-		(property "Footprint" "Custom:SW_choc_v1v2_HS_MBK"
+		(property "Footprint" "Custom:Choc_v2_PG1353_socket"
 			(at 194.31 130.81 0)
 			(effects
@@
 			)
 		)
-		(property "Footprint" "Custom:SW_choc_v1v2_HS_MBK"
+		(property "Footprint" "Custom:Choc_v2_PG1353_socket"
 			(at 99.06 110.49 0)
 			(effects
@@
 			)
 		)
-		(property "Footprint" "Custom:SW_choc_v1v2_HS_MBK"
+		(property "Footprint" "Custom:Choc_v2_PG1353_socket"
 			(at 31.75 69.85 0)
 			(effects
@@
 			)
 		)
-		(property "Footprint" "Custom:SW_choc_v1v2_HS_MBK"
+		(property "Footprint" "Custom:Choc_v2_PG1353_socket"
 			(at 60.96 110.49 0)
 			(effects
@@
 			)
 		)
-		(property "Footprint" "Custom:SW_choc_v1v2_HS_MBK"
+		(property "Footprint" "Custom:Choc_v2_PG1353_socket"
 			(at 250.19 68.58 0)
 			(effects
@@
 			)
 		)
-		(property "Footprint" "Custom:SW_choc_v1v2_HS_MBK"
+		(property "Footprint" "Custom:Choc_v2_PG1353_socket"
 			(at 60.96 90.17 0)
 			(effects
@@
 			)
 		)
-		(property "Footprint" "Custom:SW_choc_v1v2_HS_MBK"
+		(property "Footprint" "Custom:Choc_v2_PG1353_socket"
 			(at 46.99 90.17 0)
 			(effects
