File: forager-pcb/forager-pcb.kicad_pcb (KiCad board)
At the start: 2 copper layers, 236.5 x 96.3 mm, 90 parts, among them J1 Conn_01x02_Pin, J2 Conn_01x02_Pin

Commit message: Add extra column and remove all traces
Parts:
- added LCH1: ChocHS, Library:SW_choc_v2_HS_MBK, B.Cu at (-107.0, -28.0)
- added LCH11: ChocHS, Library:SW_choc_v2_HS_MBK, B.Cu at (-107.0, 6.00)
- added LCH6: ChocHS, Library:SW_choc_v2_HS_MBK, B.Cu at (-107.0, -11.0)
- added LD1: D, Diode_SMD:D_SOD-123, F.Cu at (2.38, 1.18)
- added LD13: D, Diode_SMD:D_SOD-123, F.Cu at (2.38, 7.88)
- added LD7: D, Diode_SMD:D_SOD-123, B.Cu at (-22.0, -26.0)
- added RCH10: ChocHS, Library:SW_choc_v2_HS_MBK, B.Cu at (107.0, -11.0)
- added RCH15: ChocHS, Library:SW_choc_v2_HS_MBK, B.Cu at (107.0, 6.00)
- added RCH5: ChocHS, Library:SW_choc_v2_HS_MBK, B.Cu at (107.0, -28.0)
- added RD12: D, Diode_SMD:D_SOD-123, F.Cu at (2.38, 14.6)
- added RD18: D, Diode_SMD:D_SOD-123, F.Cu at (2.38, 17.9)
- added RD6: D, Diode_SMD:D_SOD-123, F.Cu at (2.38, 11.2)
- LCH10: renamed from LCH8; footprint Custom:SW_choc_v1_HS_MBK -> Library:SW_choc_v2_HS_MBK
- LCH11: renamed from LCH9; footprint Custom:SW_choc_v1_HS_MBK -> Library:SW_choc_v2_HS_MBK
- LCH12: renamed from LCH10; footprint Custom:SW_choc_v1_HS_MBK -> Library:SW_choc_v2_HS_MBK
- LCH14: renamed from LCH11; footprint Custom:SW_choc_v1_HS_MBK -> Library:SW_choc_v2_HS_MBK
- LCH15: renamed from LCH12; footprint Custom:SW_choc_v1_HS_MBK -> Library:SW_choc_v2_HS_MBK
- LCH16: renamed from LCH13; footprint Custom:SW_choc_v1_HS_MBK -> Library:SW_choc_v2_HS_MBK
- LCH17: renamed from LCH14; footprint Custom:SW_choc_v1_HS_MBK -> Library:SW_choc_v2_HS_MBK
- LCH18: renamed from LCH15; footprint Custom:SW_choc_v1_HS_MBK -> Library:SW_choc_v2_HS_MBK
- LCH19: renamed from LCH16; footprint Custom:SW_choc_v1_HS_MBK -> Library:SW_choc_v2_HS_MBK
- LCH2: renamed from LCH1; footprint Custom:SW_choc_v1_HS_MBK -> Library:SW_choc_v2_HS_MBK
- LCH20: renamed from LCH17; footprint Custom:SW_choc_v1_HS_MBK -> Library:SW_choc_v2_HS_MBK
- LCH3: renamed from LCH2; footprint Custom:SW_choc_v1_HS_MBK -> Library:SW_choc_v2_HS_MBK
- LCH4: renamed from LCH3; footprint Custom:SW_choc_v1_HS_MBK -> Library:SW_choc_v2_HS_MBK
- LCH5: renamed from LCH4; footprint Custom:SW_choc_v1_HS_MBK -> Library:SW_choc_v2_HS_MBK
- LCH6: renamed from LCH5; footprint Custom:SW_choc_v1_HS_MBK -> Library:SW_choc_v2_HS_MBK
- LCH8: renamed from LCH6; footprint Custom:SW_choc_v1_HS_MBK -> Library:SW_choc_v2_HS_MBK
- LCH9: renamed from LCH7; footprint Custom:SW_choc_v1_HS_MBK -> Library:SW_choc_v2_HS_MBK
- RCH1, RCH2, RCH3, RCH4, RCH5: footprint Custom:SW_choc_v1_HS_MBK -> Library:SW_choc_v2_HS_MBK
- RCH10: renamed from RCH9; footprint Custom:SW_choc_v1_HS_MBK -> Library:SW_choc_v2_HS_MBK
- RCH11: renamed from RCH10; footprint Custom:SW_choc_v1_HS_MBK -> Library:SW_choc_v2_HS_MBK
- RCH13: renamed from RCH11; footprint Custom:SW_choc_v1_HS_MBK -> Library:SW_choc_v2_HS_MBK
- RCH14: renamed from RCH12; footprint Custom:SW_choc_v1_HS_MBK -> Library:SW_choc_v2_HS_MBK
- RCH15: renamed from RCH13; footprint Custom:SW_choc_v1_HS_MBK -> Library:SW_choc_v2_HS_MBK
- RCH16: renamed from RCH14; footprint Custom:SW_choc_v1_HS_MBK -> Library:SW_choc_v2_HS_MBK
- RCH17: renamed from RCH15; footprint Custom:SW_choc_v1_HS_MBK -> Library:SW_choc_v2_HS_MBK
- RCH19: renamed from RCH16; footprint Custom:SW_choc_v1_HS_MBK -> Library:SW_choc_v2_HS_MBK
- RCH20: renamed from RCH17; footprint Custom:SW_choc_v1_HS_MBK -> Library:SW_choc_v2_HS_MBK
- RCH7: renamed from RCH6; footprint Custom:SW_choc_v1_HS_MBK -> Library:SW_choc_v2_HS_MBK
- RCH8: renamed from RCH7; footprint Custom:SW_choc_v1_HS_MBK -> Library:SW_choc_v2_HS_MBK
- RCH9: renamed from RCH8; footprint Custom:SW_choc_v1_HS_MBK -> Library:SW_choc_v2_HS_MBK
- moved LCH14 18.0 mm to (-125.0, 6.00)
- moved LCH2 18.0 mm to (-125.0, -28.0)
- moved LCH8 18.0 mm to (-125.0, -11.0)
- moved LU1 18.0 mm to (-125.5, -40.0)
- moved RCH11 18.0 mm to (125.0, -11.0)
- moved RCH17 18.0 mm to (125.0, 6.00)
- moved RCH5 18.0 mm to (125.0, -28.0)
- moved REF** 18.0 mm to (-111.2, -45.8)
- moved REF** 18.0 mm to (111.2, 12.8)
- moved REF** 18.0 mm to (-111.2, 12.8)
- moved RU1 18.0 mm to (125.5, -40.0)
- renumbered LD8 to LD10, LD9 to LD11, LD10 to LD12, LD11 to LD14, LD12 to LD15, LD13 to LD16, LD14 to LD17, LD15 to LD18, LD16 to LD19, LD1 to LD2, LD17 to LD20, LD2 to LD3, LD3 to LD4, LD4 to LD5, LD5 to LD6, LD6 to LD8, LD7 to LD9, RD9 to RD10, RD10 to RD11, RD11 to RD13, RD12 to RD14, RD13 to RD15, RD14 to RD16, RD15 to RD17, RD16 to RD19, RD17 to RD20, RD6 to RD7, RD7 to RD8, RD8 to RD9, TP3 to TP2, TP2 to TP3
Connections:
- LCH10 pad 1: /LCOL2 -> /LCOL3
- LCH11 pad 1: /LCOL3 -> /LCOL4
- LCH12 pad 1: /LCOL4 -> /LCOL5
- LCH14 pad 1: /LCOL0 -> /LCOL1
- LCH15 pad 1: /LCOL1 -> /LCOL2
- LCH16 pad 1: /LCOL2 -> /LCOL3
- LCH17 pad 1: /LCOL3 -> /LCOL4
- LCH18 pad 1: /LCOL4 -> /LCOL5
- LCH19 pad 1: /LCOL3 -> /LCOL4
- LCH2 pad 1: /LCOL0 -> /LCOL1
- LCH20 pad 1: /LCOL4 -> /LCOL5
- LCH3 pad 1: /LCOL1 -> /LCOL2
- LCH4 pad 1: /LCOL2 -> /LCOL3
- LCH5 pad 1: /LCOL3 -> /LCOL4
- LCH6 pad 1: /LCOL4 -> /LCOL5
- LCH8 pad 1: /LCOL0 -> /LCOL1
- LCH9 pad 1: /LCOL1 -> /LCOL2
- LU1 pad 11: unconnected-(LU1-P1.15/10-Pad11) -> /LROW0
- LU1 pad 12: /LROW3 -> /LROW1
- LU1 pad 13: /LROW1 -> /LROW2
- LU1 pad 14: /LROW2 -> /LROW3
- LU1 pad 6: unconnected-(LU1-P0.05/5-Pad6) -> /LCOL5
- LU1 pad 7: /LROW0 -> unconnected-(LU1-P1.11/6-Pad7)
- RCH1 pad 1: /RCOL4 -> /RCOL5
- RCH10 pad 1: /RCOL1 -> /RCOL2
- RCH11 pad 1: /RCOL0 -> /RCOL1
- RCH13 pad 1: /RCOL4 -> /RCOL5
- RCH14 pad 1: /RCOL3 -> /RCOL4
- RCH15 pad 1: /RCOL2 -> /RCOL3
- RCH16 pad 1: /RCOL1 -> /RCOL2
- RCH17 pad 1: /RCOL0 -> /RCOL1
- RCH19 pad 1: /RCOL4 -> /RCOL5
- RCH2 pad 1: /RCOL3 -> /RCOL4
- RCH20 pad 1: /RCOL3 -> /RCOL4
- RCH3 pad 1: /RCOL2 -> /RCOL3
- RCH4 pad 1: /RCOL1 -> /RCOL2
- RCH5 pad 1: /RCOL0 -> /RCOL1
- RCH7 pad 1: /RCOL4 -> /RCOL5
- RCH8 pad 1: /RCOL3 -> /RCOL4
- RCH9 pad 1: /RCOL2 -> /RCOL3
- RU1 pad 1: /RROW3 -> /RCOL0
- RU1 pad 11: /RCOL3 -> /RROW0
- RU1 pad 12: /RCOL4 -> /RROW1
- RU1 pad 13: /RROW1 -> /RROW2
- RU1 pad 14: /RROW0 -> /RROW3
- RU1 pad 2: /RROW2 -> /RCOL1
- RU1 pad 3: /RCOL0 -> /RCOL2
- RU1 pad 4: /RCOL1 -> /RCOL3
- RU1 pad 5: /RCOL2 -> /RCOL4
- RU1 pad 6: unconnected-(RU1-P0.05/5-Pad6) -> /RCOL5
Routing:
- net /LROW3: track 159.1 -> 0.00 mm
- net /RCOL4: track 156.1 -> 0.00 mm, vias 1 -> 0
- net /LCOL4: track 153.3 -> 0.00 mm, vias 1 -> 0
- net /LROW1: track 136.9 -> 0.00 mm
- net /RCOL3: track 135.8 -> 0.00 mm, vias 1 -> 0
- net /LCOL3: track 133.6 -> 0.00 mm, vias 1 -> 0
- net /RROW2: track 113.4 -> 0.00 mm
- net /RROW3: track 110.5 -> 0.00 mm
- net /LCOL2: track 97.2 -> 0.00 mm, vias 1 -> 0
- net Net-(LD8-A): track 91.4 -> 0.00 mm
- net LBAT: track 90.7 -> 0.00 mm
- net /LROW2: track 84.9 -> 0.00 mm, vias 2 -> 0
- net RBAT: track 83.9 -> 0.00 mm
- net /LCOL1: track 82.1 -> 0.00 mm, vias 1 -> 0
- net /RCOL2: track 76.3 -> 0.00 mm, vias 1 -> 0
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Other:
- board size 236.5 x 96.3 mm -> 272.5 x 96.3 mm

Commit message: Giving up on meaningful commit breakdown
Parts:
- moved REF** 18.0 mm to (111.2, -45.8)
- moved LCH1 3.00 mm to (-107.0, -31.0)
- moved LCH11 3.00 mm to (-107.0, 3.00)
- moved LCH6 3.00 mm to (-107.0, -14.0)
- moved RCH10 3.00 mm to (107.0, -14.0)
- moved RCH15 3.00 mm to (107.0, 3.00)
- moved RCH5 3.00 mm to (107.0, -31.0)
- moved LCH15 1.00 mm to (-89.0, -1.00)
- moved LCH3 1.00 mm to (-89.0, -35.0)
- moved LCH9 1.00 mm to (-89.0, -18.0)
- moved RCH10 1.00 mm to (89.0, -18.0)
- moved RCH16 1.00 mm to (89.0, -1.00)
- moved RCH4 1.00 mm to (89.0, -35.0)
